Commit message: Added instruction

File: src/tresgdl_description/urdf/3gdl-control.xacro (robot description, xacro)
@@ -27,5 +27,5 @@
       <origin rpy="0 0 0" xyz="0 0 ${0.5*l}"/>
       <geometry>
-        <cylinder length="${l}" radius="${r}"/>
+        <cylinder length="${0.8*l}" radius="${r}"/>
       </geometry>
     </visual>
@@ -33,5 +33,5 @@
       <origin rpy="0 0 0" xyz="0 0 ${0.5*l}"/>
       <geometry>
-        <cylinder length="${l}" radius="${r}"/>
+        <cylinder length="${0.6*l}" radius="${r}"/>
       </geometry>
     </collision>
@@ -44,5 +44,5 @@
   <link name="world"/>
   <link name="base_link">
-    <xacro:linkcylinder m="1" l="${l0}" r="${r}"/>
+    <xacro:linkcylinder m="1" l="${l0}" r="${1.6*r}"/>
   </link>
   <link name="link_one">
@@ -69,5 +69,5 @@
     <parent link="link_one"/>
     <child link="link_two"/>
-    <origin rpy="0 0 0 " xyz="0 -${2.2*r} ${l1}"/>
+    <origin rpy="0 0 0 " xyz="0 0 ${l1}"/>
     <axis xyz="0 1 0"/>
   </joint>
@@ -75,5 +75,5 @@
     <parent link="link_two"/>
     <child link="link_three"/>
-    <origin rpy="0 ${0.5*PI} 0 " xyz="0 ${2.2*r} ${l2}"/>
+    <origin rpy="0 ${0.5*PI} 0 " xyz="0 0 ${l2}"/>
     <axis xyz="0 1 0"/>
   </joint>

Commit message: update

File: src/tresgdl_description/urdf/3gdl-control.xacro (robot description, xacro)
@@ -55,4 +55,27 @@
     <xacro:linkcylinder m="1" l="${l3}" r="${r}"/>
   </link>
+   <link name="gripper_one">
+     <inertial>
+        <origin xyz="0 0 0.05" rpy="0 0 0"/>
+     <mass value="0.05"/>
+     <inertia ixx="100"  ixy="0"  ixz="0" iyy="100" iyz="0" izz="100" />
+   </inertial>
+   <visual>
+        <origin xyz="0 0 0.05" rpy="0 0 0"/>
+      <geometry>
+       <box size="0.02 0.04 0.1" />
+     </geometry>
+     <material name="Cyan">
+       <color rgba="0 1.0 1.0 1.0"/>
+     </material>
+   </visual>
+   <collision>
+     <origin xyz="0 0 0" rpy="0 0 0"/>
+        <origin xyz="0 0 0.05" rpy="0 0 0"/>
+      <geometry>
+       <box size="0.02 0.04 0.1" />
+     </geometry>
+   </collision>
+  </link>
   <joint name="world_to_base" type="fixed">
     <parent link="world"/>
@@ -77,4 +100,11 @@
     <origin rpy="0 ${0.5*PI} 0 " xyz="0 0 ${l2}"/>
     <axis xyz="0 1 0"/>
+  </joint>
+  <joint name="arm_to_gripper_one" type="prismatic">
+    <parent link="link_three"/>
+    <child link="gripper_one"/>
+    <origin rpy="0 0 0 " xyz="0.00 -0.05 ${l3}"/>
+    <axis xyz="0 1 0"/>
+    <limit lower="0" upper="0.03" effort="10" velocity="0.5"/>
   </joint>
     <transmission name="tran1">
@@ -108,4 +138,14 @@
     </actuator>
   </transmission>
+    <transmission name="trang1">
+    <type>transmission_interface/SimpleTransmission</type>
+    <joint name="arm_to_gripper_one">
+      <hardwareInterface>hardware_interface/EffortJointInterface</hardwareInterface>
+    </joint>
+    <actuator name="motor4">
+      <hardwareInterface>hardware_interface/EffortJointInterface</hardwareInterface>
+      <mechanicalReduction>1</mechanicalReduction>
+    </actuator>
+  </transmission>
   <gazebo reference="link_two">
     <material>Gazebo/Blue</material>

Commit message: almost working gripper

File: src/tresgdl_description/urdf/3gdl-control.xacro (robot description, xacro)
@@ -64,5 +64,5 @@
         <origin xyz="0 0 0.05" rpy="0 0 0"/>
       <geometry>
-       <box size="0.02 0.04 0.1" />
+       <box size="0.05 0.02 0.1" />
      </geometry>
      <material name="Cyan">
@@ -74,5 +74,28 @@
         <origin xyz="0 0 0.05" rpy="0 0 0"/>
       <geometry>
-       <box size="0.02 0.04 0.1" />
+       <box size="0.05 0.02 0.1" />
+     </geometry>
+   </collision>
+  </link>
+   <link name="gripper_two">
+     <inertial>
+        <origin xyz="0 0 0.05" rpy="0 0 0"/>
+     <mass value="0.05"/>
+     <inertia ixx="100"  ixy="0"  ixz="0" iyy="100" iyz="0" izz="100" />
+   </inertial>
+   <visual>
+        <origin xyz="0 0 0.05" rpy="0 0 0"/>
+      <geometry>
+       <box size="0.05 0.02 0.1" />
+     </geometry>
+     <material name="Cyan">
+       <color rgba="0 1.0 1.0 1.0"/>
+     </material>
+   </visual>
+   <collision>
+     <origin xyz="0 0 0" rpy="0 0 0"/>
+        <origin xyz="0 0 0.05" rpy="0 0 0"/>
+      <geometry>
+       <box size="0.05 0.02 0.1" />
      </geometry>
    </collision>
@@ -108,4 +131,11 @@
     <limit lower="0" upper="0.03" effort="10" velocity="0.5"/>
   </joint>
+  <joint name="arm_to_gripper_two" type="prismatic">
+    <parent link="link_three"/>
+    <child link="gripper_two"/>
+    <origin rpy="0 0 0 " xyz="0.00 0.05 ${l3}"/>
+    <axis xyz="0 -1 0"/>
+    <limit lower="0" upper="0.03" effort="10" velocity="0.5"/>
+  </joint>
     <transmission name="tran1">
     <type>transmission_interface/SimpleTransmission</type>
@@ -144,4 +174,14 @@
     </joint>
     <actuator name="motor4">
+      <hardwareInterface>hardware_interface/EffortJointInterface</hardwareInterface>
+      <mechanicalReduction>1</mechanicalReduction>
+    </actuator>
+  </transmission>
+    <transmission name="trang2">
+    <type>transmission_interface/SimpleTransmission</type>
+    <joint name="arm_to_gripper_two">
+      <hardwareInterface>hardware_interface/EffortJointInterface</hardwareInterface>
+    </joint>
+    <actuator name="motor5">
       <hardwareInterface>hardware_interface/EffortJointInterface</hardwareInterface>
       <mechanicalReduction>1</mechanicalReduction>
